File: paw3395 breakout board.kicad_pcb (KiCad board)
At the start: 2 copper layers, 8.9 x 15.9 mm, 28 parts, among them J1 Conn_01x06_Socket, U1 paw3395, U2 TPS73601DBV, U3 TPS73601DBV

Commit message: Add files via upload
Parts:
- J1: footprint Connector_PinSocket_1.00mm:PinSocket_1x06_P1.00mm_Vertical -> Connector_PinSocket_2.54mm:PinSocket_1x06_P2.54mm_Vertical
- U1: footprint motion sensor:PMW3360 -> PixArt Motion Sensors:PMW3360
- moved C9 41.3 mm to (113.1, 103.4), turned to 180 degrees
- moved U2 35.1 mm to (118.1, 98.8), turned to 0 degrees
- moved C8 32.4 mm to (112.9, 98.7), turned to 90 degrees
- moved C10 31.4 mm to (117.6, 122.1), turned to -90 degrees
- moved U3 30.9 mm to (122.2, 122.1), turned to 0 degrees
- moved R4 28.9 mm to (131.2, 98.7), turned to -90 degrees
- moved R5 28.2 mm to (123.3, 98.8)
- moved C14 27.4 mm to (127.3, 98.7), turned to -90 degrees
- moved C13 26.1 mm to (130.4, 118.7), turned to 0 degrees
- moved R3 24.4 mm to (135.1, 122.0), turned to -90 degrees
- moved R1 24.3 mm to (130.3, 106.2), turned to 180 degrees
- moved R6 24.0 mm to (127.3, 122.0), turned to -90 degrees
- moved C12 20.5 mm to (131.3, 122.0), turned to -90 degrees
- moved R2 20.0 mm to (130.3, 111.1), turned to 180 degrees
- moved D3 19.7 mm to (130.3, 115.8), turned to 0 degrees
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Connections:
- C1 pad 2: GND -> GNDREF
- C2 pad 2: GND -> GNDREF
- C7 pad 1: GND -> GNDREF
- U1 pad 3: GND -> GNDREF
Routing:
- net VDD: track 0.00 -> 63.8 mm
- net GNDREF: track 0.00 -> 62.7 mm, vias 0 -> 12
- net 3V3: track 0.00 -> 58.3 mm
- net 1V9: track 0.00 -> 46.8 mm, vias 0 -> 4
- net Net-(U2-FB): track 0.00 -> 12.0 mm
- net Net-(U3-FB): track 0.00 -> 11.9 mm
- net NCS: track 0.00 -> 9.45 mm
- net MISO: track 0.00 -> 8.93 mm
- net SCLK: track 0.00 -> 8.59 mm
- net MOSI: track 0.00 -> 8.33 mm
- net Net-(U1-LED_P): track 0.00 -> 1.97 mm
- added copper zone on B.Cu, net GNDREF
Other:
- board size 8.9 x 15.9 mm -> 30 x 30.2 mm
