File: paw3395 breakout board.kicad_sch (KiCad schematic)
At the start: 28 parts, among them J1 Conn_01x06_Socket, U1 paw3395, U2 TPS73601DBV, U3 TPS73601DBV

Commit message: Add files via upload
Parts:
- J1: footprint Connector_PinSocket_1.00mm:PinSocket_1x06_P1.00mm_Vertical -> Connector_PinSocket_2.54mm:PinSocket_1x06_P2.54mm_Vertical
- U1: footprint motion sensor:PMW3360 -> PixArt Motion Sensors:PMW3360
Connections:
- net GND is gone; now on net GNDREF: C1.2, C2.2, C7.1, U1.3 (GND)
- no-connect marks 2 -> 6
